File: ElectronicsLabLamp.kicad_sch (KiCad schematic)
At the start: 0 parts

Commit message: rough sketch
Parts:
- added C1, C4: 10uF, Capacitor_SMD:C_1210_3225Metric_Pad1.33x2.70mm_HandSolder, symbol Device:C
- added C2, C3: 0.1uF, Package_TO_SOT_SMD:SOT-23-6, symbol Device:C
- added D1: LED, symbol Device:LED
- added L1: L, symbol Device:L
- added R1: R, symbol Device:R
- added U2: TPS92200D1DDC, Package_TO_SOT_SMD:SOT-23-6, symbol Driver_LED:TPS92200D1DDC
Connections:
- new net: C4.1, D1.2 (A), L1.2
- new net: D1.1 (K), R1.1, U2.1 (FB)
- new net: C3.2, L1.1, U2.6 (BOOT)
- new net: C3.1, U2.5 (SW)
- new net +12V: C1.1, C2.1, U2.4 (VIN)
- new net GND: C1.2, C2.2, C4.2, R1.2, U2.3 (GND)

Commit message: finished schematic with parts
Parts:
- L1: value L -> 8.2uH; footprint (none) -> Inductor_SMD:L_7.3x7.3_H4.5
- R1: value R -> 120mR; footprint (none) -> Resistor_SMD:R_2512_6332Metric_Pad1.40x3.35mm_HandSolder
Other:
- moved on the sheet: C1, C2
Changed lines of the file:
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@@
 	(paper "A4")
 	(junction
-		(at 97.79 86.36)
+		(at 93.98 86.36)
 		(diameter 0)
 		(color 0 0 0 0)
@@
 	)
 	(junction
-		(at 97.79 101.6)
+		(at 93.98 101.6)
 		(diameter 0)
 		(color 0 0 0 0)
 	)
 	(junction
-		(at 107.95 86.36)
+		(at 105.41 86.36)
 		(diameter 0)
 		(color 0 0 0 0)
 	)
 	(junction
-		(at 107.95 101.6)
+		(at 105.41 101.6)
 		(diameter 0)
 		(color 0 0 0 0)
@@
 	(wire
 		(pts
-			(xy 107.95 93.98) (xy 107.95 101.6)
-		)
-		(stroke
-			(width 0)
-			(type default)
-		)
-	)
-	(wire
-		(pts
-			(xy 97.79 101.6) (xy 107.95 101.6)
-		)
-		(stroke
-			(width 0)
-			(type default)
-		)
-	)
-	(wire
-		(pts
-			(xy 97.79 86.36) (xy 107.95 86.36)
+			(xy 105.41 93.98) (xy 105.41 101.6)
 		)
 		(stroke
@@
 	(wire
 		(pts
-			(xy 107.95 101.6) (xy 124.46 101.6)
-		)
-		(stroke
-			(width 0)
-			(type default)
-		)
-	)
-	(wire
-		(pts
 			(xy 134.62 91.44) (xy 151.13 91.44)
 		)
@@
 	(wire
 		(pts
-			(xy 97.79 101.6) (xy 97.79 93.98)
+			(xy 93.98 101.6) (xy 93.98 93.98)
 		)
 		(stroke
@@
 	(wire
 		(pts
-			(xy 93.98 101.6) (xy 97.79 101.6)
+			(xy 87.63 101.6) (xy 124.46 101.6)
 		)
 		(stroke
@@
 	(wire
 		(pts
-			(xy 93.98 86.36) (xy 97.79 86.36)
+			(xy 87.63 86.36) (xy 114.3 86.36)
 		)
 		(stroke
@@
 		(pts
 			(xy 158.75 86.36) (xy 165.1 86.36)
-		)
-		(stroke
-			(width 0)
-			(type default)
-		)
-	)
-	(wire
-		(pts
-			(xy 107.95 86.36) (xy 114.3 86.36)
 		)
 		(stroke
@@
 			)
 		)
-		(property "Value" "R"
+		(property "Value" "120mR"
 			(at 167.64 115.5699 0)
 			(show_name no)
@@
 			)
 		)
-		(property "Footprint" ""
+		(property "Footprint" "Resistor_SMD:R_2512_6332Metric_Pad1.40x3.35mm_HandSolder"
 			(at 163.322 114.3 90)
 			(hide yes)
@@
 	(symbol
 		(lib_id "power:+12V")
-		(at 93.98 86.36 0)
+		(at 87.63 86.36 0)
 		(unit 1)
 		(body_style 1)
@@
 		(fields_autoplaced yes)
 		(property "Reference" "#PWR01"
-			(at 93.98 90.17 0)
+			(at 87.63 90.17 0)
 			(hide yes)
 			(show_name no)
@@
 		)
 		(property "Value" "+12V"
-			(at 93.98 81.28 0)
+			(at 87.63 81.28 0)
 			(show_name no)
 			(do_not_autoplace no)
@@
 		)
 		(property "Footprint" ""
-			(at 93.98 86.36 0)
+			(at 87.63 86.36 0)
 			(hide yes)
 			(show_name no)
@@
 		)
 		(property "Datasheet" ""
-			(at 93.98 86.36 0)
+			(at 87.63 86.36 0)
 			(hide yes)
 			(show_name no)
@@
 		)
 		(property "Description" "Power symbol creates a global label with name \"+12V\""
-			(at 93.98 86.36 0)
+			(at 87.63 86.36 0)
 			(hide yes)
 			(show_name no)
@@
 			)
 		)
-		(property "Value" "L"
+		(property "Value" "8.2uH"
 			(at 154.94 83.82 90)
 			(show_name no)
@@
 			)
 		)
-		(property "Footprint" ""
+		(property "Footprint" "Inductor_SMD:L_7.3x7.3_H4.5"
 			(at 154.94 86.36 0)
 			(hide yes)
@@
 	(symbol
 		(lib_id "Device:C")
-		(at 97.79 90.17 0)
+		(at 93.98 90.17 0)
 		(unit 1)
 		(body_style 1)
@@
 		(fields_autoplaced yes)
 		(property "Reference" "C1"
-			(at 101.6 88.8999 0)
+			(at 97.79 88.8999 0)
 			(show_name no)
 			(do_not_autoplace no)
@@
 		)
 		(property "Value" "10uF"
-			(at 101.6 91.4399 0)
+			(at 97.79 91.4399 0)
 			(show_name no)
 			(do_not_autoplace no)
@@
 		)
 		(property "Footprint" "Capacitor_SMD:C_1210_3225Metric_Pad1.33x2.70mm_HandSolder"
-			(at 98.7552 93.98 0)
+			(at 94.9452 93.98 0)
 			(hide yes)
 			(show_name no)
@@
 		)
 		(property "Datasheet" ""
-			(at 97.79 90.17 0)
+			(at 93.98 90.17 0)
 			(hide yes)
 			(show_name no)
@@
 		)
 		(property "Description" "Unpolarized capacitor"
-			(at 97.79 90.17 0)
+			(at 93.98 90.17 0)
 			(hide yes)
 			(show_name no)
@@
 	(symbol
 		(lib_id "Device:C")
-		(at 107.95 90.17 0)
+		(at 105.41 90.17 0)
 		(unit 1)
 		(body_style 1)
@@
 		(fields_autoplaced yes)
 		(property "Reference" "C2"
-			(at 111.76 88.8999 0)
+			(at 109.22 88.8999 0)
 			(show_name no)
 			(do_not_autoplace no)
@@
 		)
 		(property "Value" "0.1uF"
-			(at 111.76 91.4399 0)
+			(at 109.22 91.4399 0)
 			(show_name no)
 			(do_not_autoplace no)
@@
 		)
 		(property "Footprint" "Package_TO_SOT_SMD:SOT-23-6"
-			(at 108.9152 93.98 0)
+			(at 106.3752 93.98 0)
 			(hide yes)
 			(show_name no)
@@
 		)
 		(property "Datasheet" ""
-			(at 107.95 90.17 0)
+			(at 105.41 90.17 0)
 			(hide yes)
 			(show_name no)
@@
 		)
 		(property "Description" "Unpolarized capacitor"
-			(at 107.95 90.17 0)
+			(at 105.41 90.17 0)
 			(hide yes)
 			(show_name no)
@@
 	(symbol
 		(lib_id "power:GND")
-		(at 93.98 101.6 0)
+		(at 87.63 101.6 0)
 		(unit 1)
 		(body_style 1)
@@
 		(fields_autoplaced yes)
 		(property "Reference" "#PWR02"
-			(at 93.98 107.95 0)
+			(at 87.63 107.95 0)
 			(hide yes)
 			(show_name no)
@@
 		)
 		(property "Value" "GND"
-			(at 93.98 106.68 0)
+			(at 87.63 106.68 0)
 			(show_name no)
 			(do_not_autoplace no)
@@
 		)
 		(property "Footprint" ""
-			(at 93.98 101.6 0)
+			(at 87.63 101.6 0)
 			(hide yes)
 			(show_name no)
@@
 		)
 		(property "Datasheet" ""
-			(at 93.98 101.6 0)
+			(at 87.63 101.6 0)
 			(hide yes)
 			(show_name no)
@@
 		)
 		(property "Description" "Power symbol creates a global label with name \"GND\" , ground"
-			(at 93.98 101.6 0)
-			(hide yes)
-			(show_name no)
+			(at 87.63 101.6 0)
+			(hide yes)
+			(show_name no)
